Commit message: fix(sim): URDF steering axis + PARALLEL/SPINNING modes (phase 4)
URDF: flip steering axis from (0,0,-1) to (0,0,1) so positive joint
command = CCW about z = left turn, matching ROS REP-103. The earlier
bootstrap rule preserving (0,0,-1) was based on an incomplete reading
of the real driver — its positive-angle convention is internal to its
kinematic math, not a physical constraint on the URDF.

Resolves the sign disagreement found in R07c where /odom and gz
ground truth reported opposite y-directions for an angular.z>0
command.

Messenger: implement PARALLEL and SPINNING motion modes.
- PARALLEL: all 4 wheels point in same direction = atan2(y, x);
  speed = sqrt(x^2+y^2). Side-slip sub-case (x=0, y!=0) steers to
  +/-pi/2 with sign chosen from last_nonzero_x to keep "forward"
  consistent.
- SPINNING: all 4 wheels tangent to a circle centered at the
  vehicle origin; wheel velocity sized to make body yaw at the
  commanded rate. Range-wrap for joint limits; per-wheel
  velocity sign-flipped on wrap.
- Kinematic models for /odom integration: ParallelModel and
  SpinningModel ports from real driver's kinematics_model.hpp.

Also fixes an inherited R07 bug in calculate_steering_angle:
ZeroDivisionError when cmd_vel has linear.x=0 (pure-spin command).
Add an early return for lin<1e-6 with (0.0, 0.0) — radius 0 forces
SPINNING mode upstream. Matches smalleha's div-by-zero guard in
the real driver (S-abk a5609b7 incorporated this on the C++ side).

All four motion modes (DUAL_ACKERMAN, PARALLEL, SPINNING,
SIDE_SLIP-via-PARALLEL) now implemented end-to-end.

File: ranger_mini_v3_description/urdf/ranger_mini_v3.xacro (robot description, xacro)
@@ -91,5 +91,5 @@
       <!-- Original used axis (0,0,-1); we keep that so positive command =
            CW seen from above, matching the real-driver kinematic model. -->
-      <axis xyz="0 0 -1"/>
+      <axis xyz="0 0 1"/>
       <limit effort="${steer_effort}" velocity="${steer_vel}"
              lower="${-steer_limit}" upper="${steer_limit}"/>
